Commit message: Update

File: packages/multi_robot_follow/urdf/red_turtlebot.urdf (robot description, URDF)
Before this commit: robot red_turtlebot, 4 links, 3 joints
Links:
- removed link caster_wheel
- link base_link: geometry collision box size=0.5 0.3 0.2; visual box size=0.5 0.3 0.2
Joints:
- removed joint caster_wheel_joint
